File: leaf/leaf/leaf.kicad_sch (KiCad schematic)
At the start: 31 parts, among them J1 52435-2471, J2 Conn_01x04, J3 Conn_01x04, J4 USB_C_Receptacle_USB2.0_16P, U1 ESP32-S3-WROOM-1, U2 USBLC6-2SC6, U3 LM1117DT-3.3

Commit message: update
Parts:
- J3: footprint (none) -> Connector_PinHeader_2.54mm:PinHeader_1x04_P2.54mm_Vertical
Other:
- moved on the sheet: J3, R1, R2
Changed lines of the file:
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@@
 	)
 	(junction
-		(at 93.98 45.72)
+		(at 96.52 30.48)
 		(diameter 0)
 		(color 0 0 0 0)
@@
 	(wire
 		(pts
-			(xy 115.57 64.77) (xy 113.03 64.77)
+			(xy 88.9 53.34) (xy 86.36 53.34)
 		)
 		(stroke
@@
 	(wire
 		(pts
-			(xy 83.82 41.91) (xy 77.47 41.91)
+			(xy 86.36 26.67) (xy 80.01 26.67)
 		)
 		(stroke
@@
 	(wire
 		(pts
-			(xy 83.82 45.72) (xy 77.47 45.72)
+			(xy 86.36 30.48) (xy 80.01 30.48)
 		)
 		(stroke
@@
 	(wire
 		(pts
-			(xy 113.03 67.31) (xy 119.38 67.31)
+			(xy 86.36 55.88) (xy 92.71 55.88)
 		)
 		(stroke
@@
 	(wire
 		(pts
-			(xy 88.9 41.91) (xy 93.98 41.91)
+			(xy 91.44 26.67) (xy 96.52 26.67)
 		)
 		(stroke
@@
 	(wire
 		(pts
-			(xy 116.84 73.66) (xy 116.84 72.39)
+			(xy 90.17 62.23) (xy 90.17 60.96)
 		)
 		(stroke
@@
 	(wire
 		(pts
-			(xy 93.98 41.91) (xy 93.98 45.72)
+			(xy 96.52 26.67) (xy 96.52 30.48)
 		)
 		(stroke
@@
 	(wire
 		(pts
-			(xy 93.98 45.72) (xy 93.98 50.8)
+			(xy 96.52 30.48) (xy 96.52 35.56)
 		)
 		(stroke
@@
 	(wire
 		(pts
-			(xy 116.84 72.39) (xy 113.03 72.39)
+			(xy 90.17 60.96) (xy 86.36 60.96)
 		)
 		(stroke
@@
 	(wire
 		(pts
-			(xy 115.57 63.5) (xy 115.57 64.77)
+			(xy 88.9 52.07) (xy 88.9 53.34)
 		)
 		(stroke
@@
 	(wire
 		(pts
-			(xy 113.03 69.85) (xy 119.38 69.85)
+			(xy 86.36 58.42) (xy 92.71 58.42)
 		)
 		(stroke
@@
 	(wire
 		(pts
-			(xy 88.9 45.72) (xy 93.98 45.72)
+			(xy 91.44 30.48) (xy 96.52 30.48)
 		)
 		(stroke
@@
 	)
 	(label "CC2"
-		(at 77.47 45.72 180)
+		(at 80.01 30.48 180)
 		(effects
 			(font
@@
 	)
 	(label "CC1"
-		(at 77.47 41.91 180)
+		(at 80.01 26.67 180)
 		(effects
 			(font
@@
 	)
 	(label "USB_D-"
-		(at 119.38 69.85 0)
+		(at 92.71 58.42 0)
 		(effects
 			(font
@@
 	)
 	(label "USB_D+"
-		(at 119.38 67.31 0)
+		(at 92.71 55.88 0)
 		(effects
 			(font
@@
 	(symbol
 		(lib_id "power:+5V")
-		(at 115.57 63.5 0)
+		(at 88.9 52.07 0)
 		(unit 1)
 		(exclude_from_sim no)
@@
 		(fields_autoplaced yes)
 		(property "Reference" "#PWR038"
-			(at 115.57 67.31 0)
+			(at 88.9 55.88 0)
 			(effects
 				(font
@@
 		)
 		(property "Value" "+5V"
-			(at 115.57 58.42 0)
+			(at 88.9 46.99 0)
 			(effects
 				(font
@@
 		)
 		(property "Footprint" ""
-			(at 115.57 63.5 0)
+			(at 88.9 52.07 0)
 			(effects
 				(font
@@
 		)
 		(property "Datasheet" ""
-			(at 115.57 63.5 0)
+			(at 88.9 52.07 0)
 			(effects
 				(font
@@
 		)
 		(property "Description" "Power symbol creates a global label with name \"+5V\""
-			(at 115.57 63.5 0)
+			(at 88.9 52.07 0)
 			(effects
 				(font
@@
 	(symbol
 		(lib_id "Device:R_Small")
-		(at 86.36 41.91 90)
+		(at 88.9 26.67 90)
 		(unit 1)
 		(exclude_from_sim no)
@@
 		(dnp no)
 		(property "Reference" "R1"
-			(at 84.836 39.37 90)
+			(at 87.376 24.13 90)
 			(effects
 				(font
@@
 		)
 		(property "Value" "5.1K"
-			(at 88.392 39.37 90)
+			(at 90.932 24.13 90)
 			(effects
 				(font
@@
 		)
 		(property "Footprint" "Resistor_SMD:R_0402_1005Metric_Pad0.72x0.64mm_HandSolder"
-			(at 86.36 41.91 0)
+			(at 88.9 26.67 0)
 			(effects
 				(font
@@
 		)
 		(property "Datasheet" "~"
-			(at 86.36 41.91 0)
+			(at 88.9 26.67 0)
 			(effects
 				(font
@@
 		)
 		(property "Description" "Resistor, small symbol"
-			(at 86.36 41.91 0)
+			(at 88.9 26.67 0)
 			(effects
 				(font
@@
 	(symbol
 		(lib_id "Device:R_Small")
-		(at 86.36 45.72 90)
+		(at 88.9 30.48 90)
 		(unit 1)
 		(exclude_from_sim no)
@@
 		(dnp no)
 		(property "Reference" "R2"
-			(at 85.09 48.26 90)
+			(at 87.63 33.02 90)
 			(effects
 				(font
@@
 		)
 		(property "Value" "5.1K"
-			(at 88.9 48.26 90)
+			(at 91.44 33.02 90)
 			(effects
 				(font
@@
 		)
 		(property "Footprint" "Resistor_SMD:R_0402_1005Metric_Pad0.72x0.64mm_HandSolder"
-			(at 86.36 45.72 0)
+			(at 88.9 30.48 0)
 			(effects
 				(font
@@
 		)
 		(property "Datasheet" "~"
-			(at 86.36 45.72 0)
+			(at 88.9 30.48 0)
 			(effects
 				(font
@@
 		)
 		(property "Description" "Resistor, small symbol"
-			(at 86.36 45.72 0)
+			(at 88.9 30.48 0)
 			(effects
 				(font
@@
 	(symbol
 		(lib_id "power:GND")
-		(at 93.98 50.8 0)
+		(at 96.52 35.56 0)
 		(unit 1)
 		(exclude_from_sim no)
@@
 		(fields_autoplaced yes)
 		(property "Reference" "#PWR011"
-			(at 93.98 57.15 0)
+			(at 96.52 41.91 0)
 			(effects
 				(font
@@
 		)
 		(property "Value" "GND"
-			(at 93.98 55.88 0)
+			(at 96.52 40.64 0)
 			(effects
 				(font
@@
 		)
 		(property "Footprint" ""
-			(at 93.98 50.8 0)
+			(at 96.52 35.56 0)
 			(effects
 				(font
@@
 		)
 		(property "Datasheet" ""
-			(at 93.98 50.8 0)
+			(at 96.52 35.56 0)
 			(effects
 				(font
@@
 		)
 		(property "Description" "Power symbol creates a global label with name \"GND\" , ground"
-			(at 93.98 50.8 0)
+			(at 96.52 35.56 0)
 			(effects
 				(font
@@
 	(symbol
 		(lib_id "Connector_Generic:Conn_01x04")
-		(at 107.95 67.31 0)
+		(at 81.28 55.88 0)
 		(mirror y)
 		(unit 1)
@@
 		(fields_autoplaced yes)
 		(property "Reference" "J3"
-			(at 107.95 60.96 0)
+			(at 81.28 49.53 0)
 			(effects
 				(font
@@
 		)
 		(property "Value" "Conn_01x04"
-			(at 107.95 60.96 0)
+			(at 81.28 49.53 0)
 			(effects
 				(font
@@
 			)
 		)
-		(property "Footprint" ""
-			(at 107.95 67.31 0)
+		(property "Footprint" "Connector_PinHeader_2.54mm:PinHeader_1x04_P2.54mm_Vertical"
+			(at 81.28 55.88 0)
 			(effects
 				(font
@@
 		)
 		(property "Datasheet" "~"
-			(at 107.95 67.31 0)
+			(at 81.28 55.88 0)
 			(effects
 				(font
@@
 		)
 		(property "Description" "Generic connector, single row, 01x04, script generated (kicad-library-utils/schlib/autogen/connector/)"
-			(at 107.95 67.31 0)
+			(at 81.28 55.88 0)
 			(effects
 				(font
@@
 	(symbol
 		(lib_id "power:GND")
-		(at 116.84 73.66 0)
+		(at 90.17 62.23 0)
 		(unit 1)
 		(exclude_from_sim no)
@@
 		(fields_autoplaced yes)
 		(property "Reference" "#PWR037"
-			(at 116.84 80.01 0)
+			(at 90.17 68.58 0)
 			(effects
 				(font
@@
 		)
 		(property "Value" "GND"
-			(at 116.84 78.74 0)
+			(at 90.17 67.31 0)
 			(effects
 				(font
@@
 		)
 		(property "Footprint" ""
-			(at 116.84 73.66 0)
+			(at 90.17 62.23 0)
 			(effects
 				(font
@@
 		)
 		(property "Datasheet" ""
-			(at 116.84 73.66 0)
+			(at 90.17 62.23 0)
 			(effects
 				(font
@@
 		)
 		(property "Description" "Power symbol creates a global label with name \"GND\" , ground"
-			(at 116.84 73.66 0)
+			(at 90.17 62.23 0)
 			(effects
 				(font
